File: PLUTO60.kicad_pcb (KiCad board)
At the start: 2 copper layers, 285 x 94.6 mm, 122 parts, among them M1 XIAO-RP2040

Commit message: Corrected MCU placement & tidied routing
Parts:
- moved D1 11.8 mm to (15.1, -78.5), turned to -90 degrees
- moved M1 9.48 mm to (40.7, -73.7)
- moved D6 7.49 mm to (49.2, -78.6), turned to 90 degrees
- moved D45 3.17 mm to (295.3, -78.6)
- moved D59 2.86 mm to (275.4, -38.9), turned to 180 degrees
- moved D58 2.25 mm to (250.0, -19.8), turned to 0 degrees
Routing:
- net COL2: track 468.4 -> 385.2 mm
- net COL4: track 411.6 -> 461.2 mm, vias 0 -> 2
- net COL1: track 260.5 -> 298.2 mm
- net COL3: track 488.6 -> 521.2 mm
- net ROW4: track 462.0 -> 488.0 mm, vias 9 -> 2
- net ROW3: track 271.2 -> 286.8 mm, vias 1 -> 2
- net ROW1: track 233.1 -> 247.8 mm, vias 1 -> 2
- net ROW2: track 257.7 -> 271.6 mm, vias 1 -> 2
- net COL0: track 226.7 -> 239.7 mm
- net COL5: track 393.9 -> 405.4 mm
- net ROW0: track 219.9 -> 227.2 mm
- net Net-(D1-Pad1): track 12.2 -> 17.2 mm
- net Net-(D6-Pad2): track 15.1 -> 10.5 mm
- net Net-(D59-Pad2): track 10.5 -> 14.3 mm
- net GND: track 0.00 -> 3.53 mm, vias 0 -> 1
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Other:
- board text added: "PLUTO60 V1.3 Designed by Morronrost"
- board text removed: "PLUTO60 V1.2 Designed by Morronrost"
